Commit message: added clibration for the base to lucid

File: lbr_description/urdf/iiwa7/iiwa7.xacro (robot description, xacro)
@@ -12,13 +12,4 @@
         name="initial_joint_positions_path"
         default="$(find lbr_description)/ros2_control/initial_joint_positions.yaml" />
-    <!-- KDL requires a link without inertia / Gazebo requires a connection to world link or robot
-    will tipple https://github.com/lbr-stack/lbr_fri_ros2_stack/issues/230 -->
-    <link name="world" />
-    <!--joint
-        between <robot_name>_world_link and robot_name_link_0-->
-    <joint name="$(arg robot_name)_world_joint" type="fixed">
-        <parent link="world" />
-        <child link="$(arg robot_name)_link_0" />
-    </joint>
     <!-- iiwa -->
     <xacro:iiwa7
